File: DAM_Circuit/DAM_Circuit.kicad_pcb (KiCad board)
At the start: 2 copper layers, 200 x 100 mm, 98 parts, among them J1 Screw_Terminal_01x02, J2 Screw_Terminal_01x02, J3 Power Source (12V), Q1 IRLZ44N, Q2 IRLZ44N, SW1 SW_Push, SW2 SW_Push, U1 74LS147, U10 74LS48, U11 74LS125, U12 74LS20, U13 74LS21, U14 74LS85, U15 74LS85, U16 74LS32, U17 A1104xLH, U18 A1104xLH, U19 A1104xLH, U2 74LS175, U20 A1104xLH, U21 A1104xLH, U22 A1104xLH, U23 A1104xLH, U24 A1104xLH, U25 A1104xLH, U26 A1104xLH, U27 SM420561N, U28 SM420561N, U29 LM7805_TO220, U3 74LS157, U4 74LS85, U5 74LS04, U6 74LS32, U7 74LS04, U8 74LS85, U9 74LS157

Commit message: 6.7.2026 time=3:33 finalized schematic position please route manually
Parts:
- moved BZ1 30.2 mm to (264.0, 94.3), turned to 180 degrees
- moved C6 21.6 mm to (164.0, 177.9), turned to 0 degrees
- moved U13 21.4 mm to (162.7, 158.7), turned to 0 degrees
- moved C14 19.3 mm to (272.5, 109.4)
- moved U10 19.3 mm to (294.1, 107.9)
- moved C7 17.1 mm to (179.8, 178.0), turned to 0 degrees
- moved C12 16.3 mm to (229.6, 94.0)
- moved U11 16.3 mm to (248.7, 92.7)
- moved C9 14.7 mm to (228.9, 109.7)
- moved U8 14.7 mm to (250.4, 108.2)
- moved U12 11.3 mm to (178.8, 158.9), turned to 0 degrees
- moved C10 10.0 mm to (272.1, 94.8)
- moved U9 10.0 mm to (293.9, 93.0)
- moved J3 7.45 mm to (109.5, 94.0)
- moved U7 6.95 mm to (214.2, 129.4)
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
Commit message: 6.7.2026 already routed, need to compress more
Parts:
- moved J3 91.0 mm to (200.5, 94.5), turned to 180 degrees
- moved U29 88.8 mm to (213.0, 93.0)
- moved C20 88.8 mm to (218.8, 103.0)
- moved C19 88.8 mm to (211.8, 103.0)
- moved C6 54.7 mm to (109.3, 176.9)
- moved U13 54.7 mm to (108.0, 157.7)
- moved C7 52.6 mm to (127.2, 177.0)
- moved U12 52.6 mm to (126.2, 157.9)
- moved C13 43.1 mm to (184.7, 176.7)
- moved U16 43.1 mm to (183.4, 157.6)
- moved C16 41.4 mm to (167.6, 178.9)
- moved U15 41.4 mm to (166.1, 157.3)
- moved C15 38.5 mm to (149.4, 179.0)
- moved U14 38.5 mm to (147.9, 157.4)
- moved R12 34.1 mm to (153.5, 110.3)
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Routing:
- net GND: track 0.00 -> 1758.0 mm, vias 0 -> 58
- net +5V: track 0.00 -> 1225.9 mm, vias 0 -> 32
- net D: track 0.00 -> 268.1 mm, vias 0 -> 9
- net B: track 0.00 -> 246.0 mm, vias 0 -> 15
- net A: track 0.00 -> 245.0 mm, vias 0 -> 13
- net Net-(U8-Oa>b): track 0.00 -> 222.6 mm, vias 0 -> 5
- net C: track 0.00 -> 183.7 mm, vias 0 -> 14
- net Net-(U11-Pad2): track 0.00 -> 169.1 mm, vias 0 -> 1
- net +12V: track 0.00 -> 161.1 mm, vias 0 -> 6
- net Net-(U13-Pad12): track 0.00 -> 147.0 mm, vias 0 -> 5
- net P10: track 0.00 -> 144.6 mm, vias 0 -> 1
- net Net-(U13-Pad9): track 0.00 -> 128.8 mm, vias 0 -> 4
- net Net-(C17-Pad1): track 0.00 -> 123.3 mm, vias 0 -> 2
- net Net-(C18-Pad1): track 0.00 -> 118.0 mm, vias 0 -> 1
- net Net-(U2-D1): track 0.00 -> 112.1 mm, vias 0 -> 5
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
Commit message: 6.7.2026 zoning is done, added drill holes, added grouping only last thing is gerber files
Parts:
- added REF**: KiCad-Logo2_6mm_SilkScreen, Symbol:KiCad-Logo2_6mm_SilkScreen, F.Cu at (204.0, 150.5)
- added REF**: MountingHole_2.2mm_M2, MountingHole:MountingHole_2.2mm_M2, F.Cu at (232.5, 106.5)
- added REF**: MountingHole_2.2mm_M2, MountingHole:MountingHole_2.2mm_M2, F.Cu at (105.0, 181.0)
- added REF**: MountingHole_2.2mm_M2, MountingHole:MountingHole_2.2mm_M2, F.Cu at (267.5, 160.5)
- added REF**: MountingHole_2.2mm_M2, MountingHole:MountingHole_2.2mm_M2, F.Cu at (297.0, 113.5)
Routing:
- net GND: track 1758.0 -> 1724.9 mm, vias 58 -> 53
- net +12V: track 161.1 -> 168.2 mm, vias 6 -> 5
- net Net-(U2-D1): track 112.1 -> 111.1 mm
- net +5V: track 1225.9 -> 1226.4 mm, vias 32 -> 29
- added copper zone on B.Cu, net (none)
- added copper zone on F.Cu, net (none)
Other:
- board text added: "+"
- board text added: "+12V"
- board text added: "+5v"
- board text added: "+IN"
- board text added: "-"
- board text added: "-IN"
- board text added: "100R"
- board text added: "104"
- board text added: "106"
- board text added: "10K"
- board text added: "10^0"
- board text added: "10^1"
- board text added: "1N4007"
- board text added: "1ST GATE"
- board text added: "2-INPUT OR GATE"
- board text added: "2ND GATE"
- board text added: "330R"
- board text added: "4-INPUT AND GATE"
- board text added: "4-INPUT NAND GATE"
- board text added: "7 SEGMENT DECODER"
- board text added: "74LS04"
- board text added: "74LS125"
- board text added: "74LS147"
- board text added: "74LS157"
- board text added: "74LS175"
- board text added: "74LS20"
- board text added: "74LS21"
- board text added: "74LS32"
- board text added: "74LS48"
- board text added: "74LS85"
- board text added: "ALARM"
- board text added: "BS ECE 2A SY 2025~2026"
- board text added: "BUZZER"
- board text added: "CPE 301 - LOGIC CIRCUITS AND SWITCHING THEORY"
- board text added: "Collaboration: Anday, John Kevin I. Aquino, Jasmine J. Haque, Majeed Mohammad P. Leonardo, John Ruiz A. Llamas, Kristyn Cayte A. Magdamit, Rovic B. Quintana, Francesca Maris S"
- board text added: "D-TYPE FLIP FLOP"
- board text added: "GND"
- board text added: "H1"
- board text added: "H10"
- board text added: "H2"
- board text added: "H3"
- board text added: "H4"
- board text added: "H5"
- board text added: "H6"
- board text added: "H7"
- board text added: "H8"
- board text added: "H9"
- board text added: "HEX INVERTER (NOT GATE)"
- board text added: "IRLZ44N"
- board text added: "L7805"
- board text added: "LCD INDICATOR AND EVENTS: 00 LEVEL - DRAINING CALIBRATION 01 LEVEL - NO EVENT 02 LEVEL - NO EVENT 03 LEVEL - NO EVENT 04 LEVEL - GREATER THAN 4 OPENS GATE 1 05 LEVEL - NO EVENT 06 LEVEL - NOTHING 07 LEVEL - NOTHING 08 LEVEL - GREATER THAN 8 OPENS GATE 2 09 LEVEL - NO EVENT 10 LEVEL - ALARM ACTIVATED"
- board text added: "LEVEL RANGE: 1 ~ 10"
- board text added: "MAGNITUDE COMPARITOR"
- board text added: "MANUAL GATE OVERRIDE"
- board text added: "MULTIPLEXER"
- board text added: "OUT"
- board text added: "POWER"
- board text added: "PRIORITY ENCODER"
- board text added: "SOLENOID"
- board text added: "TRI-STATE BUFFER"
- board text added: "The PCB serves as the central hardware controller for an automated dam spillway system, processing inputs from 10 Hall Effect sensors through a priority encoder and combinational logic to manage two solenoid valves. Additionally, the board drivesa 7-segment display forreal-time water level monitoring and triggers a continuous emergency alarm at critical thresholds, providing a complete discrete d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"
- board text added: "WATER LEVEL"
- board text added: "这块PCB作为自动化大坝溢洪系统的中央硬件控制器，通过优先编码器和组合逻辑处理来自10 个霍尔效应传感器的输入，以控制两个电磁阀。此外，该电路板驱动7段数码管进行实时水位监测， 并在达到临界水位时触发持续的紧急警报，提供了一个完整的分立数字逻辑解决方案。"
